Commit message: Addition of camera and LiDAR
Addition of the camera and LiDAR sensors to the robot, the parameter of the robot standing are yet to be tuned

File: Robot/unitree_ros/robots/a1_description/xacro/gazebo.xacro (robot description, xacro)
@@ -249,3 +249,83 @@
         <kd  value="1.0"/>
     </gazebo>
+    <!-- camera -->
+  <gazebo reference="camera_link">
+    <sensor type="camera" name="camera1">
+      <update_rate>30.0</update_rate>
+      <camera name="head">
+        <horizontal_fov>1.3962634</horizontal_fov>
+        <image>
+          <width>800</width>
+          <height>800</height>
+          <format>R8G8B8</format>
+        </image>
+        <clip>
+          <near>0.02</near>
+          <far>300</far>
+        </clip>
+		<noise>
+          <type>gaussian</type>
+          <mean>0.0</mean>
+          <stddev>0.007</stddev>
+        </noise>
+      </camera>
+      <plugin name="camera_controller" filename="libgazebo_ros_camera.so">
+        <alwaysOn>true</alwaysOn>
+        <updateRate>0.0</updateRate>
+        <cameraName>camera1</cameraName>
+        <imageTopicName>image_raw</imageTopicName>
+        <cameraInfoTopicName>camera_info</cameraInfoTopicName>
+        <frameName>camera_link</frameName>
+        <hackBaseline>0.07</hackBaseline>
+        <distortionK1>0.0</distortionK1>
+        <distortionK2>0.0</distortionK2>
+        <distortionK3>0.0</distortionK3>
+        <distortionT1>0.0</distortionT1>
+        <distortionT2>0.0</distortionT2>
+      </plugin>
+    </sensor>
+  </gazebo>
+	<!-- LiDAR -->
+      <gazebo reference="vlp16_link">
+	      <turnGravityOff>true</turnGravityOff>
+	      <sensor name='velodyne-VLP16' type='ray'>
+	          <visualize>0</visualize>
+	          <update_rate>1</update_rate>
+	          <ray>
+	            <scan>
+	              <horizontal>
+	                <samples>1800</samples>
+	                <resolution>1</resolution>
+	                <min_angle>-3.14159</min_angle>
+	                <max_angle>+3.14159</max_angle>
+	              </horizontal>
+	              <vertical>
+	                <samples>16</samples>
+	                <resolution>1</resolution>
+	                <min_angle>-0.261799</min_angle>
+	                <max_angle>0.261799</max_angle>
+	              </vertical>
+	            </scan>
+	            <range>
+	              <min>0.055</min>
+	              <max>70</max>
+	              <resolution>0.001</resolution>
+	            </range>
+	            <noise>
+	              <type>gaussian</type>
+	              <mean>0</mean>
+	              <stddev>0</stddev>
+	            </noise>
+	          </ray>
+	          <plugin name='gazebo_ros_laser_controller' filename='libgazebo_ros_velodyne_laser.so'>
+	            <topicName>/vlp16_points</topicName>
+	            <frameName>vlp16_link</frameName>
+	            <min_range>0.9</min_range>
+	            <max_range>70.0</max_range>
+	            <gaussianNoise>0.008</gaussianNoise>
+	            <robotNamespace>/</robotNamespace>
+	          </plugin>
+	          <pose frame=''>0 0 0 0 0 0</pose>
+	        </sensor>
+	    </gazebo>
 </robot>

File: Robot/unitree_ros/robots/a1_description/xacro/robot.xacro (robot description, xacro)
@@ -6,4 +6,5 @@
     <xacro:include filename="$(find a1_description)/xacro/stairs.xacro"/>
     <xacro:include filename="$(find a1_description)/xacro/gazebo.xacro"/>
+    <xacro:include filename="$(find a1_description)/../velodyne_VLP16/vlp16.urdf.xacro"/>
     <!-- <xacro:include filename="$(find a1_gazebo)/launch/stairs.urdf.xacro"/> -->
     <!-- <xacro:stairs stairs="15" xpos="0" ypos="0" zpos="0" /> -->
@@ -122,3 +123,42 @@
     </xacro:leg>
     <!-- <xacro:stairs stairs="15" xpos="0" ypos="2.0" zpos="0" /> -->
+    <link name="camera_link">
+	    <collision>
+	      <origin xyz="-0.2 0 0.05" rpy="0 0 0"/>
+	      <geometry>
+		<box size="0.01 0.02 0.01"/>
+	      </geometry>
+	    </collision>
+	    <visual>
+	      <origin xyz="0 0 0" rpy="0 0 0"/>
+	      <geometry>
+		<box size="0.01 0.02 0.01"/>
+	      </geometry>
+	      <material name="gray"/>
+	    </visual>
+	    <inertial>
+	      <mass value="1" />
+	      <origin xyz="0 0 0" rpy="0 0 0"/>
+	      <inertia ixx="1e-6" ixy="0" ixz="0" iyy="1" iyz="0" izz="1e-6" />
+	    </inertial>
+  </link>
+  <joint name="camera_joint" type="fixed">
+	    <axis xyz="1 0 0" />
+	    <origin xyz="${trunk_length} 0 0" rpy="0 0 0"/>
+	    <parent link="trunk"/>
+	    <child link="camera_link"/>
+   </joint>
+   <!-- LIDAR -->
+   <xacro:arg name="xyz" default="0.2 0 0.09" />
+   <xacro:arg name="rpy" default="0 0 0" />
+   <xacro:arg name="noise" default="0.008" />
+   <xacro:arg name="min_angle" default="-180" />
+   <xacro:arg name="max_angle" default="180" />
+   <xacro:arg name="azimuth" default="0.2" />
+   <xacro:arg name="hz" default="1" />
+   <xacro:arg name="lidar_name" default="vlp16" />
+   <vlp16 parent="trunk" name="$(arg lidar_name)" hz="$(arg hz)" noise="$(arg noise)"
+     min_angle="$(arg min_angle)" max_angle="$(arg max_angle)" azimuth="$(arg azimuth)">
+     <origin xyz="$(arg xyz)" rpy="$(arg rpy)"/>
+   </vlp16>
 </robot>
